File: hardware/driver_board/driver_board.kicad_pcb (KiCad board)
At the start: 2 copper layers, 68.6 x 53.3 mm, 8 parts, among them P1 Power, P2 Analog, P3 Digital, P4 Digital, P5 CONN_01X01, P6 CONN_01X01, P7 CONN_01X01, P8 CONN_01X01

Commit message: Finished rev1 PCBs
Parts:
- added C1: 0.1uF, Capacitors_SMD:C_0805, F.Cu at (132.0, 91.4)
- added C2: 1uF, Capacitors_SMD:C_0805, F.Cu at (128.8, 91.4)
- added C3: 220uF, Capacitors_THT:CP_Radial_D8.0mm_P3.80mm, F.Cu at (128.8, 112.4)
- added F1: Fuse, Fuse_Holders_and_Fuses:Fuse_SMD1206_HandSoldering, F.Cu at (131.3, 103.5)
- added J1: BARREL_JACK, matthew:Kobiconn_163-179PH-EX, B.Cu at (111.0, 102.2)
- added J2: CONN_01X03, Pin_Headers:Pin_Header_Straight_1x03_Pitch2.54mm, F.Cu at (173.9, 83.2)
- added J3: CONN_01X06, matthew:Molex_53047_0610, F.Cu at (173.2, 114.3)
- added Q1: Q_NMOS_GDS, TO_SOT_Packages_SMD:TO-263-3_TabPin2, F.Cu at (149.1, 95.9)
- added Q2: Q_NMOS_GDS, TO_SOT_Packages_SMD:TO-263-3_TabPin2, F.Cu at (163.1, 95.9)
- added R1: 10KR, Resistors_SMD:R_0805, F.Cu at (138.3, 84.5)
- added R2: 10KR, Resistors_SMD:R_0805, F.Cu at (134.5, 84.5)
- added U1: MIC4124, SMD_Packages:SOIC-8-N, F.Cu at (137.7, 91.4)
Connections:
- P1 pad 8: /Vin -> VCC
- P3 pad 1: /A5(SCL) -> /A5(SCL)_2
- P3 pad 2: /A4(SDA) -> /A4(SDA)_2
Routing:
- net VCC: track 0.00 -> 121.1 mm, vias 0 -> 2
- net Net-(Q2-Pad1): track 0.00 -> 40.2 mm, vias 0 -> 2
- net GND: track 0.00 -> 38.2 mm, vias 0 -> 3
- net /C_LED: track 0.00 -> 36.3 mm
- net +5V: track 0.00 -> 25.2 mm
- net /W_LED: track 0.00 -> 24.2 mm
- net /10(**/SS): track 0.00 -> 22.5 mm
- net /9(**): track 0.00 -> 20.4 mm
- net Net-(Q1-Pad1): track 0.00 -> 17.4 mm
- net /A0: track 0.00 -> 12.2 mm
- net /A1: track 0.00 -> 11.7 mm
- net /A2: track 0.00 -> 11.1 mm
- net /A3: track 0.00 -> 10.6 mm
- net Net-(F1-Pad2): track 0.00 -> 8.12 mm
- added copper zone on B.Cu, net GND
Other:
- board text added: "UnnaturalLight (driver board) - Rev 1"
