File: hardware/driver_board/driver_board.kicad_pcb (KiCad board)
At the start: 2 copper layers, 68.6 x 53.3 mm, 20 parts, among them J1 BARREL_JACK, J2 CONN_01X03, J3 CONN_01X06, P1 Power, P2 Analog, P3 Digital, P4 Digital, P5 CONN_01X01, P6 CONN_01X01, P7 CONN_01X01, P8 CONN_01X01, Q1 Q_NMOS_GDS, Q2 Q_NMOS_GDS, U1 MIC4124

Commit message: Added fab files
Other:
- rule pad_to_mask_clearance: 0 -> 0.1016
Changed lines of the file:
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@@
     (pad_size 4.064 4.064)
     (pad_drill 3.048)
-    (pad_to_mask_clearance 0)
+    (pad_to_mask_clearance 0.1016)
+    (pad_to_paste_clearance -0.127)
     (aux_axis_origin 110.998 126.365)
     (grid_origin 110.998 126.365)
     (visible_elements FFFFFF7F)
     (pcbplotparams
-      (layerselection 0x00030_80000001)
-      (usegerberextensions false)
-      (excludeedgelayer true)
+      (layerselection 0x010f0_80000001)
+      (usegerberextensions true)
+      (excludeedgelayer false)
       (linewidth 0.100000)
       (plotframeref false)
@@
       (outputformat 1)
       (mirror false)
-      (drillshape 1)
+      (drillshape 0)
       (scaleselection 1)
-      (outputdirectory ""))
+      (outputdirectory fab/))
   )
   (net 0 "")
