File: hardware/ui_board/ui_board.kicad_pcb (KiCad board)
At the start: 2 copper layers, 64 x 18.5 mm, 5 parts, among them J1 CONN_01X06, SW1 SW_SPST

Commit message: Added fab files
Other:
- rule pad_to_mask_clearance: 0.2 -> 0.1016
Changed lines of the file:
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@@
     (pad_size 2.5 2.5)
     (pad_drill 1.3)
-    (pad_to_mask_clearance 0.2)
+    (pad_to_mask_clearance 0.1016)
+    (pad_to_paste_clearance -0.127)
     (aux_axis_origin 0 0)
     (visible_elements FFFFFF7F)
     (pcbplotparams
-      (layerselection 0x00030_80000001)
-      (usegerberextensions false)
-      (excludeedgelayer true)
+      (layerselection 0x010f0_80000001)
+      (usegerberextensions true)
+      (excludeedgelayer false)
       (linewidth 0.100000)
       (plotframeref false)
@@
       (outputformat 1)
       (mirror false)
-      (drillshape 1)
+      (drillshape 0)
       (scaleselection 1)
-      (outputdirectory ""))
+      (outputdirectory fab/))
   )
   (net 0 "")
